Commit message: New updates....

File: new_mod/urdf/new_mod.urdf (robot description, URDF)
Before this commit: robot new_mod, 8 links, 7 joints
Links:
- link end_effector: geometry collision mesh filename=package://new_mod/meshes/end_effector2.obj; visual mesh filename=package://new_mod/meshes/end_effector2.obj
